Commit message: I fixed the discontinuity in position of the robot in RVIZ!! I had both the joint state publisher and the robot state publisher running. This seems to be an issue. I talked to Michael and he said he turned his joint state publsiher off for this too. I should read up on a lot of the ROS tools. I have a shaky understanding of a lot them

File: src/nuturtle_description/urdf/diff_drive.urdf.xacro (robot description, xacro)
@@ -11,16 +11,4 @@
 <xacro:property name="chassis_thickness" value="${props['chassis_thickness']}" />
 <xacro:property name="caster_radius" value="${(wheel_radius - (chassis_thickness/2.0)) / 2}" />
-<!-- slidebot is a robot that has 1 linear and 1 rotational degree of freedom -->
-<!-- The base from which the body slides -->
-<link name="world" >
-	<visual>
-		<geometry>
-			<sphere radius="0.01" />
-		</geometry>
-		<material name="green_mat">
-			<color rgba="0 1 0 1" />
-		</material>
-	</visual>
-</link>
 <!-- the movable body -->
 <link name="base_link">
@@ -68,11 +56,4 @@
 	</visual>
 </link>
-<!-- The joints -->
-<!-- Link body to base frame -->
-  <joint name="world_base" type="fixed">
-	  <origin xyz="0 0 ${wheel_radius}" rpy="0 0 0" />
-	  <parent link="world"/>
-	  <child link="base_link"/>
-  </joint>
   <!-- Link body to base frame -->
   <joint name="base_caster" type="fixed">
@@ -81,5 +62,5 @@
           <child link="caster"/>
   </joint>
-  <joint name="left_wheel_axle" type="revolute">
+  <joint name="left_wheel_axle" type="continuous">
 	  <origin xyz="0.0 ${wheel_base/2} 0.0" rpy="0 0 0" />
 	  <axis xyz = "0 1 0" />
@@ -88,5 +69,5 @@
 	  <limit velocity="1.0" effort="10" lower="0" upper="180"/>
   </joint>
-  <joint name="right_wheel_axle" type="revolute">
+  <joint name="right_wheel_axle" type="continuous">
 	  <origin xyz="0.0 ${-1 * wheel_base/2} 0.0" rpy="0 0 0" />
 	  <axis xyz = "0 1 0" />

Commit message: I fixed the bug that was causing the robot's caster to go through the ground/not detect collisions. I also changed the colors of the robot in gazebo. She's a pretty robot now!

File: src/nuturtle_description/urdf/diff_drive.urdf.xacro (robot description, xacro)
@@ -10,5 +10,8 @@
 <xacro:property name="chassis_length" value="${props['chassis_length']}" />
 <xacro:property name="chassis_thickness" value="${props['chassis_thickness']}" />
-<xacro:property name="caster_radius" value="${(wheel_radius - (chassis_thickness/2.0)) / 2}" />
+<xacro:property name="wheel_axle_offset" value="${props['wheel_axle_offset']}" />
+<xacro:property name="caster_radius" value="${wheel_axle_offset/2}" />
+<xacro:property name="lidar_radius" value="${props['lidar_radius']}" />
+<xacro:property name="lidar_height" value="${props['lidar_height']}" />
 <!-- the movable body -->
 <link name="base_link">
@@ -22,4 +25,29 @@
 		<origin rpy="0 0 0" xyz="${chassis_length/2 - wheel_radius} 0.0 0.0"/>
 	</visual>
+	<inertial>
+      		<origin rpy="0 0 0" xyz="${chassis_length/2 - wheel_radius} 0.0 0.0"/>
+      		<mass value = "1.0"/>
+		<inertia ixx="${(1/12)*(chassis_thickness**2 + wheel_base**2)}"
+			iyy="${(1/12) * (chassis_thickness**2 + chassis_length**2)}"
+			izz="${(1/12)*(chassis_length**2 + wheel_base**2)}" ixy="0"
+			ixz="0" iyz="0"/>
+    	</inertial>
+	<collision>
+      		<origin rpy="0 0 0" xyz="${chassis_length/2 - wheel_radius} 0.0 0.0"/>
+    	  	<geometry>
+        		<box size="${chassis_length} ${wheel_base} ${chassis_thickness}" />
+     		</geometry>
+	</collision>
+</link>
+<link name="base_scan">
+        <visual>
+                <origin xyz="0.0 0.0 0.0" rpy="0.0 0.0 0" />
+                <geometry>
+			<cylinder radius="${lidar_radius}" length="${lidar_height}" />
+                </geometry>
+                <material name="red_mat">
+                        <color rgba="0 0 1 0.4" />
+                </material>
+        </visual>
 </link>
 <link name="caster">
@@ -32,9 +60,23 @@
                 </material>
                 <origin rpy="0 0 0" xyz="0.0 0.0 0.0"/>
-        </visual>
+	</visual>
+	<collision>
+		<geometry>
+                        <sphere radius="${caster_radius}" />
+                </geometry>
+                <origin rpy="0 0 0" xyz="0.0 0.0 0.0"/>
+	</collision>
+	<inertial>
+                <origin rpy="0 0 0" xyz="0.0 0.0 0.0"/>
+                <mass value = "0.1"/>
+		<inertia ixx="${0.40 * 0.1 * caster_radius*caster_radius}"
+			 iyy="${0.40 * 0.1 * caster_radius*caster_radius}"
+			 izz="${0.40 * 0.1 * caster_radius*caster_radius}"
+			 ixy="0" ixz="0" iyz="0"/>
+        </inertial>
 </link>
 <link name="left_wheel">
 	<visual>
-		<origin xyz="0.0 0.0 0.0" rpy="${3.14/2} 0.0 0" />
+		<origin xyz="0.0 ${wheel_width/2} 0.0" rpy="${3.14/2} 0.0 0" />
 		<geometry>
 			<cylinder radius="${wheel_radius}" length="${wheel_width}" />
@@ -44,8 +86,21 @@
 		</material>
 	</visual>
+	<inertial>
+		<origin xyz="0.0 ${wheel_width/2} 0.0" rpy="${3.14/2} 0.0 0"/>
+		<mass value="0.1"/>
+		<inertia ixx="${(1/12)*0.1*(3 * wheel_radius**2 + wheel_width**2)}" iyy="${.5 * 0.1 * wheel_radius**2}"
+			izz="${(1/12)*0.1*(3*wheel_radius**2+wheel_width**2)}" ixy="0"
+			ixz="0" iyz="0"/>
+	</inertial>
+	<collision>
+        	<origin xyz="0.0 ${wheel_width/2} 0.0" rpy="${3.14/2} 0.0 0"/>
+        	<geometry>
+            		<cylinder radius="${wheel_radius}" length="${wheel_width}" />
+       		</geometry>
+      	</collision>
 </link>
 <link name="right_wheel">
 	<visual>
-		<origin xyz="0.0 0.0 0.0" rpy="${3.14/2} 0.0 0.0" />
+		<origin xyz="0.0 ${-1 * wheel_width/2} 0.0" rpy="${3.14/2} 0.0 0.0" />
 		<geometry>
 			<cylinder radius="${wheel_radius}" length="${wheel_width}" />
@@ -55,13 +110,26 @@
 		</material>
 	</visual>
+	<inertial>
+                <origin xyz="0.0 ${-1 * wheel_width/2} 0.0" rpy="${3.14/2} 0.0 0.0"/>
+		<mass value="0.1"/>
+		<inertia ixx="${(1/12)*0.1*(3 * wheel_radius**2 + wheel_width**2)}" iyy="${.5 * 0.1 * wheel_radius**2}"
+			izz="${(1/12)*0.1*(3*wheel_radius**2+wheel_width**2)}"
+			ixy="0" ixz="0" iyz="0"/>
+        </inertial>
+	<collision>
+                <origin xyz="0.0 ${-1 * wheel_width/2} 0.0" rpy="${3.14/2} 0.0 0.0"/>
+                <geometry>
+                        <cylinder radius="${wheel_radius}" length="${wheel_width}" />
+                </geometry>
+        </collision>
 </link>
   <!-- Link body to base frame -->
   <joint name="base_caster" type="fixed">
-	  <origin xyz="${ (-1 * wheel_radius + chassis_length) - (caster_radius)  } 0 ${(-1 * wheel_radius) + (wheel_radius - chassis_thickness/2.0) / 2.0}" rpy="0 0 0" />
+	  <origin xyz="${ (-1 * wheel_radius + chassis_length) - (caster_radius) } 0.0 ${(-1 * chassis_thickness/2) - caster_radius}" rpy="0 0 0" />
           <parent link="base_link"/>
-          <child link="caster"/>
+	  <child link="caster"/>
   </joint>
   <joint name="left_wheel_axle" type="continuous">
-	  <origin xyz="0.0 ${wheel_base/2} 0.0" rpy="0 0 0" />
+	  <origin xyz="0.0 ${wheel_base/2} ${-1 * wheel_radius - wheel_axle_offset}" rpy="0 0 0" />
 	  <axis xyz = "0 1 0" />
 	  <parent link="base_link" />
@@ -70,5 +138,5 @@
   </joint>
   <joint name="right_wheel_axle" type="continuous">
-	  <origin xyz="0.0 ${-1 * wheel_base/2} 0.0" rpy="0 0 0" />
+	  <origin xyz="0.0 ${-1 * wheel_base/2} ${-1 * wheel_radius - wheel_axle_offset}" rpy="0 0 0" />
 	  <axis xyz = "0 1 0" />
 	  <parent link="base_link" />
@@ -76,3 +144,10 @@
 	  <limit velocity="1.0" effort="10" lower="0" upper="180"/>
   </joint>
+  <joint name="base_scanner" type="fixed">
+	  <origin xyz="0.0 0.0 ${lidar_height/2 + chassis_thickness/2}" rpy="0 0 0" />
+          <axis xyz = "0 1 0" />
+          <parent link="base_link" />
+          <child link="base_scan" />
+          <limit velocity="1.0" effort="10" lower="0" upper="180"/>
+  </joint>
 </robot>
