Commit message: Starting to tune the PID controller in gazebo

File: src/nuturtle_gazebo/urdf/diff_drive.gazebo.xacro (robot description, xacro)
@@ -2,4 +2,21 @@
 <robot xmlns:xacro="http://www.ros.org/wiki/xacro" name="diff_drive" >
 <xacro:include filename="$(find nuturtle_description)/urdf/diff_drive.urdf.xacro" />
+<xacro:property name="yaml_file" value="$(find nuturtle_description)/config/diff_params.yaml" />
+<xacro:property name="props" value="${load_yaml(yaml_file)}"/>
+<xacro:property name="encoder_ticks_per_revolution" value="${props['encoder_ticks_per_revolution']}" />
+<xacro:property name="motor_power" value="${props['motor_power']}" />
+<xacro:property name="motor_torque" value="${props['motor_torque']}" />
+<xacro:property name="left_wheel_joint" value="${props['left_wheel_joint']}" />
+<xacro:property name="right_wheel_joint" value="${props['right_wheel_joint']}" />
+<gazebo>
+	<plugin name="turtle_drive_plugin" filename="/home/peter/Desktop/Turtlebot/catkin_ws/devel/lib/libturtle_drive_plugin.so">
+		<sensor_frequency>200.0</sensor_frequency>
+		<encoder_ticks_per_revolution>${encoder_ticks_per_revolution}</encoder_ticks_per_revolution>
+		<motor_power>${motor_power}</motor_power>
+		<motor_torque>${motor_torque}</motor_torque>
+		<left_wheel_joint>${left_wheel_joint}</left_wheel_joint>
+		<right_wheel_joint>${right_wheel_joint}</right_wheel_joint>
+	</plugin>
+</gazebo>
 <gazebo reference="base_link">
 	<material>Gazebo/BlueLaser</material>
@@ -10,6 +27,6 @@
 <gazebo reference="caster">
     <material>Gazebo/DarkGrey</material>
-    <mu1>0.1</mu1>
-    <mu2>0.1</mu2>
+    <mu1>0.01</mu1>
+    <mu2>0.01</mu2>
     <minDepth>0.001</minDepth>
     <maxVel>1.0</maxVel>

Commit message: I added the laser scanner to the robot's .gazebo.urdf and also cleaned up some git issues. Yikes, it looks like I wasn't tracking a few files but now I am

File: src/nuturtle_gazebo/urdf/diff_drive.gazebo.xacro (robot description, xacro)
@@ -54,3 +54,35 @@
    <kd>10</kd>
 </gazebo>
+<gazebo reference="base_scan">
+  <material>Gazebo/FlatBlack</material>
+  <sensor type="ray" name="lds_lfcd_sensor">
+    <pose>0 0 0 0 0 0</pose>
+    <visualize>true</visualize>
+    <update_rate>5</update_rate>
+    <ray>
+      <scan>
+        <horizontal>
+          <samples>360</samples>
+          <resolution>1</resolution>
+          <min_angle>0.0</min_angle>
+          <max_angle>6.28319</max_angle>
+        </horizontal>
+      </scan>
+      <range>
+        <min>0.120</min>
+        <max>3.5</max>
+        <resolution>0.015</resolution>
+      </range>
+      <noise>
+        <type>gaussian</type>
+        <mean>0.0</mean>
+        <stddev>0.01</stddev>
+      </noise>
+    </ray>
+    <plugin name="gazebo_ros_lds_lfcd_controller" filename="libgazebo_ros_laser.so">
+      <topicName>scan</topicName>
+      <frameName>base_scan</frameName>
+    </plugin>
+  </sensor>
+</gazebo>
 </robot>
